Commit message: initial commit

File: os_robots_description/urdf/backup_urdf_gazebo/tw_base_v1.gazebo.xacro (robot description, xacro)
@@ -5,5 +5,5 @@
     </gazebo>
     <gazebo reference="n20-43mm-d-shaft-wheel-1.snapshot.9_2"><!--wheel_left_link>-->
-        <!-- <mu1>0.1</mu1>
+        <mu1>0.1</mu1>
         <mu2>0.1</mu2>
         <kp>500000.0</kp>
@@ -11,9 +11,9 @@
         <minDepth>0.001</minDepth>
         <maxVel>0.1</maxVel>
-        <fdir1>1 0 0</fdir1> -->
+        <fdir1>1 0 0</fdir1>
         <material>Gazebo/FlatBlack</material>
     </gazebo>
     <gazebo reference="n20-43mm-d-shaft-wheel-1.snapshot.9"><!--wheel_right_link-->
-        <!-- <mu1>0.1</mu1>
+        <mu1>0.1</mu1>
         <mu2>0.1</mu2>
         <kp>500000.0</kp>
@@ -21,23 +21,23 @@
         <minDepth>0.001</minDepth>
         <maxVel>0.1</maxVel>
-        <fdir1>1 0 0</fdir1> -->
+        <fdir1>1 0 0</fdir1>
         <material>Gazebo/FlatBlack</material>
     </gazebo>
     <gazebo reference="ball">
-        <!-- <mu1>0.1</mu1>
+        <mu1>0.1</mu1>
         <mu2>0.1</mu2>
         <kp>1000000.0</kp>
         <kd>100.0</kd>
         <minDepth>0.001</minDepth>
-        <maxVel>1.0</maxVel> -->
+        <maxVel>1.0</maxVel>
         <material>Gazebo/FlatBlack</material>
     </gazebo>
     <gazebo reference="ball_2">
-        <!-- <mu1>0.1</mu1>
+        <mu1>0.1</mu1>
         <mu2>0.1</mu2>
         <kp>1000000.0</kp>
         <kd>100.0</kd>
         <minDepth>0.001</minDepth>
-        <maxVel>1.0</maxVel> -->
+        <maxVel>1.0</maxVel>
         <material>Gazebo/FlatBlack</material>
     </gazebo>
@@ -53,5 +53,5 @@
         <publishTf>true</publishTf>
         <publishWheelJointState>true</publishWheelJointState>
-        <legacyMode>true</legacyMode>
+        <legacyMode>false</legacyMode>
         <updateRate>30</updateRate>
         <leftJoint>LM_Revolute</leftJoint>

File: os_robots_description/urdf/backup_urdf_gazebo/tw_base_v1.urdf.xacro (robot description, xacro)
@@ -19,5 +19,5 @@
         <origin xyz= "-0.000128133 -9.90901e-05 0.0147895" rpy="1.69309e-15 6.93889e-18 -6.04901e-16" />
     <geometry>
-            <mesh filename="package://os_robots_description/meshes/backup/v1/part_1.stl"/>
+            <mesh filename="package://os_robots_description/meshes/part_1.stl"/>
     </geometry>
     <material name="part_1_material">
@@ -28,5 +28,5 @@
         <origin xyz="-0.000128133 -9.90901e-05 0.0147895" rpy="1.69309e-15 6.93889e-18 -6.04901e-16" />
     <geometry>
-        <mesh filename="package://os_robots_description/meshes/backup/v1/part_1.stl"/>
+        <mesh filename="package://os_robots_description/meshes/part_1.stl"/>
     </geometry>
     <material name="part_1_material">
@@ -44,5 +44,5 @@
         <origin xyz="0.127619 0.231707 0.00135678" rpy="3.14159 2.65197e-31 0" />
     <geometry>
-        <mesh filename="package://os_robots_description/meshes/backup/v1/n@).stl"/>
+        <mesh filename="package://os_robots_description/meshes/n@).stl"/>
     </geometry>
     <material name="n@)_material">
@@ -53,5 +53,5 @@
         <origin xyz="0.127619 0.231707 0.00135678" rpy="3.14159 2.65197e-31 0" />
     <geometry>
-        <mesh filename="package://os_robots_description/meshes/backup/v1/n@).stl"/>
+        <mesh filename="package://os_robots_description/meshes/n@).stl"/>
     </geometry>
     <material name="n@)_material">
@@ -69,5 +69,5 @@
         <origin xyz="-0.0365766 0.030151 0.0172766" rpy="3.14159 9.86076e-32 0" />
     <geometry>
-        <mesh filename="package://os_robots_description/meshes/backup/v1/n20-43mm-d-shaft-wheel-1.snapshot.9.stl"/>
+        <mesh filename="package://os_robots_description/meshes/n20-43mm-d-shaft-wheel-1.snapshot.9.stl"/>
     </geometry>
     <material name="n20-43mm-d-shaft-wheel-1.snapshot.9_material">
@@ -76,7 +76,7 @@
     </visual>
     <collision>
-        <origin xyz="-0.0365766 0.030151 0.0172766" rpy="3.14159 9.86076e-32 0" /><!--3.14159 9.86076e-32 0-->
-    <geometry>
-        <mesh filename="package://os_robots_description/meshes/backup/v1/n20-43mm-d-shaft-wheel-1.snapshot.9.stl"/>
+        <origin xyz="-0.0365766 0.030151 0.0172766" rpy="0 0 0" /><!--3.14159 9.86076e-32 0-->
+    <geometry>
+        <cylinder length="0.018" radius="0.0215"/><!--<mesh filename="package://os_robots_description/meshes/n20-43mm-d-shaft-wheel-1.snapshot.9.stl"/>-->
     </geometry>
     <material name="n20-43mm-d-shaft-wheel-1.snapshot.9_material">
@@ -95,5 +95,5 @@
 <child link="n20-43mm-d-shaft-wheel-1.snapshot.9" />
 <axis xyz="0 0 1"/>
-<limit effort="100" velocity="100" />
+<limit effort="1" velocity="20" />
 <joint_properties friction="0.0"/>
 </joint>
@@ -121,5 +121,5 @@
         <origin xyz="0.127619 0.231707 0.00135678" rpy="3.14159 2.65197e-31 0" />
     <geometry>
-        <mesh filename="package://os_robots_description/meshes/backup/v1/n@).stl"/>
+        <mesh filename="package://os_robots_description/meshes/n@).stl"/>
     </geometry>
     <material name="n@)_material">
@@ -130,5 +130,5 @@
         <origin xyz="0.127619 0.231707 0.00135678" rpy="3.14159 2.65197e-31 0" />
     <geometry>
-        <mesh filename="package://os_robots_description/meshes/backup/v1/n@).stl"/>
+        <mesh filename="package://os_robots_description/meshes/n@).stl"/>
     </geometry>
     <material name="n@)_material">
@@ -146,5 +146,5 @@
         <origin xyz="-0.0365766 0.030151 0.0172766" rpy= "-3.14159 1.63787e-47 0"/> <!--"-3.14159 1.63787e-47 0"-->
     <geometry>
-        <mesh filename="package://os_robots_description/meshes/backup/v1/n20-43mm-d-shaft-wheel-1.snapshot.9.stl"/>
+        <mesh filename="package://os_robots_description/meshes/n20-43mm-d-shaft-wheel-1.snapshot.9.stl"/>
     </geometry>
     <material name="n20-43mm-d-shaft-wheel-1.snapshot.9_material">
@@ -153,7 +153,7 @@
     </visual>
     <collision>
-        <origin xyz="-0.0365766 0.030151 0.0172766" rpy= "-3.14159 1.63787e-47 0"/><!--"-3.14159 1.63787e-47 0"-->
-    <geometry>
-        <mesh filename="package://os_robots_description/meshes/backup/v1/n20-43mm-d-shaft-wheel-1.snapshot.9.stl"/>
+        <origin xyz="-0.0365766 0.030151 0.0172766" rpy= "0 0 0"/><!--"-3.14159 1.63787e-47 0"-->
+    <geometry>
+         <cylinder length="0.018" radius="0.0215"/><!--<mesh filename="package://os_robots_description/meshes/n20-43mm-d-shaft-wheel-1.snapshot.9.stl"/>-->
     </geometry>
     <material name="n20-43mm-d-shaft-wheel-1.snapshot.9_material">
@@ -171,6 +171,6 @@
 <parent link="n@)_2" />
 <child link="n20-43mm-d-shaft-wheel-1.snapshot.9_2" />
-<axis xyz="0 0 -1"/>
-<limit effort="100" velocity="100"/>
+<axis xyz="0 0 1"/>
+<limit effort="1" velocity="20"/>
 <joint_properties friction="0.0"/>
 </joint>
@@ -198,5 +198,5 @@
         <origin xyz="0 0 0" rpy="-1.5708 -0 0" />
     <geometry>
-        <mesh filename="package://os_robots_description/meshes/backup/v1/wheel''s_body.stl"/>
+        <mesh filename="package://os_robots_description/meshes/wheel''s_body.stl"/>
     </geometry>
     <material name="wheel''s_body_material">
@@ -207,5 +207,5 @@
         <origin xyz="0 0 0" rpy="-1.5708 -0 0" />
     <geometry>
-        <mesh filename="package://os_robots_description/meshes/backup/v1/wheel''s_body.stl"/>
+        <mesh filename="package://os_robots_description/meshes/wheel''s_body.stl"/>
     </geometry>
     <material name="wheel''s_body_material">
@@ -223,5 +223,5 @@
         <origin xyz="0 0 0" rpy="0 -0 0" />
     <geometry>
-        <mesh filename="package://os_robots_description/meshes/backup/v1/ball.stl"/>
+        <mesh filename="package://os_robots_description/meshes/ball.stl"/>
     </geometry>
     <material name="ball_material">
@@ -232,5 +232,5 @@
         <origin xyz="0 0 0" rpy="0 -0 0" />
     <geometry>
-        <mesh filename="package://os_robots_description/meshes/backup/v1/ball.stl"/>
+        <mesh filename="package://os_robots_description/meshes/ball.stl"/>
     </geometry>
     <material name="ball_material">
@@ -264,5 +264,5 @@
         <origin xyz="0 0 0" rpy="-1.5708 -0 0" />
     <geometry>
-        <mesh filename="package://os_robots_description/meshes/backup/v1/wheel''s_body.stl"/>
+        <mesh filename="package://os_robots_description/meshes/wheel''s_body.stl"/>
     </geometry>
     <material name="wheel''s_body_material">
@@ -273,5 +273,5 @@
         <origin xyz="0 0 0" rpy="-1.5708 -0 0" />
     <geometry>
-        <mesh filename="package://os_robots_description/meshes/backup/v1/wheel''s_body.stl"/>
+        <mesh filename="package://os_robots_description/meshes/wheel''s_body.stl"/>
     </geometry>
     <material name="wheel''s_body_material">
@@ -289,5 +289,5 @@
         <origin xyz="0 0 0" rpy="0 -0 0" />
     <geometry>
-        <mesh filename="package://os_robots_description/meshes/backup/v1/ball.stl"/>
+        <mesh filename="package://os_robots_description/meshes/ball.stl"/>
     </geometry>
     <material name="ball_material">
@@ -298,5 +298,5 @@
         <origin xyz="0 0 0" rpy="0 -0 0" />
     <geometry>
-        <mesh filename="package://os_robots_description/meshes/backup/v1/ball.stl"/>
+        <mesh filename="package://os_robots_description/meshes/ball.stl"/>
     </geometry>
     <material name="ball_material">

File: os_robots_description/urdf/tw_base_v2.gazebo.xacro (robot description, xacro)
@@ -1,47 +1,21 @@
 <?xml version="1.0"?>
-<robot name="tw_base_v1_sim" xmlns:xacro="http://ros.org/wiki/xacro">
+<robot name="tw_base_v2_sim" xmlns:xacro="http://ros.org/wiki/xacro">
     <gazebo reference="part_1"><!--base_link-->
         <material>Gazebo/DarkGrey</material>
     </gazebo>
     <gazebo reference="n20-43mm-d-shaft-wheel-1.snapshot.9_2"><!--wheel_left_link>-->
-        <!-- <mu1>0.1</mu1>
-        <mu2>0.1</mu2>
-        <kp>500000.0</kp>
-        <kd>10.0</kd>
-        <minDepth>0.001</minDepth>
-        <maxVel>0.1</maxVel>
-        <fdir1>1 0 0</fdir1> -->
         <material>Gazebo/FlatBlack</material>
     </gazebo>
     <gazebo reference="n20-43mm-d-shaft-wheel-1.snapshot.9"><!--wheel_right_link-->
-        <!-- <mu1>0.1</mu1>
-        <mu2>0.1</mu2>
-        <kp>500000.0</kp>
-        <kd>10.0</kd>
-        <minDepth>0.001</minDepth>
-        <maxVel>0.1</maxVel>
-        <fdir1>1 0 0</fdir1> -->
         <material>Gazebo/FlatBlack</material>
     </gazebo>
     <gazebo reference="ball">
-        <!-- <mu1>0.1</mu1>
-        <mu2>0.1</mu2>
-        <kp>1000000.0</kp>
-        <kd>100.0</kd>
-        <minDepth>0.001</minDepth>
-        <maxVel>1.0</maxVel> -->
         <material>Gazebo/FlatBlack</material>
     </gazebo>
     <gazebo reference="ball_2">
-        <!-- <mu1>0.1</mu1>
-        <mu2>0.1</mu2>
-        <kp>1000000.0</kp>
-        <kd>100.0</kd>
-        <minDepth>0.001</minDepth>
-        <maxVel>1.0</maxVel> -->
         <material>Gazebo/FlatBlack</material>
     </gazebo>
     <gazebo>
-        <plugin name="tw_base_v1_controller" filename="libgazebo_ros_diff_drive.so">
+        <plugin name="tw_base_v2_controller" filename="libgazebo_ros_diff_drive.so">
         <commandTopic>cmd_vel</commandTopic>
         <odometryTopic>odom</odometryTopic>

File: os_robots_description/urdf/tw_base_v3.gazebo.xacro (robot description, xacro)
@@ -1,47 +1,21 @@
 <?xml version="1.0"?>
-<robot name="tw_base_v1_sim" xmlns:xacro="http://ros.org/wiki/xacro">
+<robot name="tw_base_v3_sim" xmlns:xacro="http://ros.org/wiki/xacro">
     <gazebo reference="part_1"><!--base_link-->
         <material>Gazebo/DarkGrey</material>
     </gazebo>
     <gazebo reference="n20-43mm-d-shaft-wheel-1.snapshot.9_2"><!--wheel_left_link>-->
-        <!-- <mu1>0.1</mu1>
-        <mu2>0.1</mu2>
-        <kp>500000.0</kp>
-        <kd>10.0</kd>
-        <minDepth>0.001</minDepth>
-        <maxVel>0.1</maxVel>
-        <fdir1>1 0 0</fdir1> -->
         <material>Gazebo/FlatBlack</material>
     </gazebo>
     <gazebo reference="n20-43mm-d-shaft-wheel-1.snapshot.9"><!--wheel_right_link-->
-        <!-- <mu1>0.1</mu1>
-        <mu2>0.1</mu2>
-        <kp>500000.0</kp>
-        <kd>10.0</kd>
-        <minDepth>0.001</minDepth>
-        <maxVel>0.1</maxVel>
-        <fdir1>1 0 0</fdir1> -->
         <material>Gazebo/FlatBlack</material>
     </gazebo>
     <gazebo reference="ball">
-        <!-- <mu1>0.1</mu1>
-        <mu2>0.1</mu2>
-        <kp>1000000.0</kp>
-        <kd>100.0</kd>
-        <minDepth>0.001</minDepth>
-        <maxVel>1.0</maxVel> -->
         <material>Gazebo/FlatBlack</material>
     </gazebo>
     <gazebo reference="ball_2">
-        <!-- <mu1>0.1</mu1>
-        <mu2>0.1</mu2>
-        <kp>1000000.0</kp>
-        <kd>100.0</kd>
-        <minDepth>0.001</minDepth>
-        <maxVel>1.0</maxVel> -->
         <material>Gazebo/FlatBlack</material>
     </gazebo>
     <gazebo>
-        <plugin name="tw_base_v1_controller" filename="libgazebo_ros_diff_drive.so">
+        <plugin name="tw_base_v3_controller" filename="libgazebo_ros_diff_drive.so">
         <commandTopic>cmd_vel</commandTopic>
         <odometryTopic>odom</odometryTopic>
